Commit message: wip

File: urdf/unit02/src/my_mira_description/urdf/mira_simple_collisions_inertias.urdf (robot description, URDF)
Before this commit: robot mira, 2 links, 1 joints
Links:
- added link camera_link, mass 0.001; visual box size=0.0005 0.0005 0.0005
- added link head_link, mass 0.02; collision sphere radius=0.06; visual sphere radius=0.06
- added link left_eye_link, mass 0.001; visual cylinder length=0.00525 radius=0.00525
- added link pitch_M2_link, mass 0.001; visual cylinder length=0.005 radius=0.01
- added link right_eye_link, mass 0.001; visual cylinder length=0.00525 radius=0.00525
- added link yaw_M3_link, mass 0.001; visual cylinder length=0.005 radius=0.01
Joints:
- added joint base_head_joint: type fixed, parent yaw_M3_link, child head_link, origin xyz=0 0 0.06 rpy=0 0 0
- added joint head_camera_joint: type fixed, parent head_link, child camera_link, origin xyz=0 0.057 0.0255 rpy=0 0 0
- added joint head_lefteye_joint: type fixed, parent head_link, child left_eye_link, origin xyz=0.0095 0.057 0.0085 rpy=-1.5708 0 0
- added joint head_righteye_joint: type fixed, parent head_link, child right_eye_link, origin xyz=-0.0095 0.057 0.0085 rpy=-1.5708 0 0
- added joint pitch_joint: type revolute, parent roll_M1_link, child pitch_M2_link, origin xyz=0 0 0 rpy=0 -1.5708 0, axis 0 1 0, limit lower=0 upper=0.44 effort=0.1 velocity=0.005
- added joint yaw_joint: type continuous, parent pitch_M2_link, child yaw_M3_link, origin xyz=0.01 0 0 rpy=0 1.5708 0, axis 0 0 1, limit effort=0.1 velocity=0.01

Commit message: wip

File: urdf/unit02/src/my_mira_description/urdf/mira_simple_collisions_inertias.urdf (robot description, URDF)
Before this commit: robot mira, 8 links, 7 joints
Links:
- removed link camera_link
- removed link head_link
- removed link left_eye_link
- removed link pitch_M2_link
- removed link right_eye_link
- removed link yaw_M3_link
Joints:
- removed joint base_head_joint
- removed joint head_camera_joint
- removed joint head_lefteye_joint
- removed joint head_righteye_joint
- removed joint pitch_joint
- removed joint yaw_joint
