Commit message: wip

File: urdf/unit02/src/my_mira_description/urdf/mira_with_controllers.urdf (robot description, URDF)
Before this commit: robot mira, 8 links, 7 joints
Links:
- link base_link: geometry collision cylinder length=0.09 radius=0.06; visual cylinder length=0.09 radius=0.06
- link head_link: geometry collision sphere radius=0.06; visual sphere radius=0.06
- link left_eye_link: geometry visual cylinder length=0.00525 radius=0.00525
- link right_eye_link: geometry visual cylinder length=0.00525 radius=0.00525

Commit message: wip

File: urdf/unit02/src/my_mira_description/urdf/mira_with_controllers.urdf (robot description, URDF)
Before this commit: robot mira, 8 links, 7 joints
Links:
- link head_link: geometry collision cylinder length=0.035 radius=0.06; visual sphere radius=0.06

Commit message: wip

File: urdf/unit02/src/my_mira_description/urdf/mira_with_controllers.urdf (robot description, URDF)
Before this commit: robot mira, 8 links, 7 joints
Links:
- link head_link: geometry collision cylinder length=0.035 radius=0.06; visual sphere radius=0.08
