Commit message: wip

File: urdf/unit02/src/my_mira_description/urdf/mira.urdf (robot description, URDF)
Before this commit: robot mira, 8 links, 7 joints
Links:
- link head_link: geometry collision sphere radius=0.08; visual sphere radius=0.06
Joints:
- joint base_head_joint: origin xyz=0 0 0 rpy=0 0 0 -> xyz=0 0 0.04 rpy=0 0 0
