Commit message: wip

File: urdf/unit03/src/my_gurdy_description/urdf/gurdy.urdf (robot description, URDF)
Before this commit: robot mira, 3 links, 1 joints
Links:
- removed link link0
- added link footM1_link; visual sphere radius=0.008
- added link footM2_link; visual sphere radius=0.008
- added link footM3_link; visual sphere radius=0.008
- added link head_link; visual mesh filename=package://my_gurdy_description/models/gurdy/meshes/gurdy_he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
- added link lowerleg_M1_link; visual mesh filename=package://my_gurdy_description/models/gurdy/meshes/gurdy_lo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
- added link lowerleg_M2_link; visual mesh filename=package://my_gurdy_description/models/gurdy/meshes/gurdy_lo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
- added link lowerleg_M3_link; visual mesh filename=package://my_gurdy_description/models/gurdy/meshes/gurdy_lo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
- added link upperleg_M1_link; visual mesh filename=package://my_gurdy_description/models/gurdy/meshes/gurdy_hi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
- added link upperleg_M2_link; visual mesh filename=package://my_gurdy_description/models/gurdy/meshes/gurdy_hi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
- added link upperleg_M3_link; visual mesh filename=package://my_gurdy_description/models/gurdy/meshes/gurdy_hi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
- link base_link: geometry 
Joints:
- added joint basefoot_peg_M1_basefoot_M1_joint_joint: type fixed, parent lowerleg_M1_link, child footM1_link, origin xyz=0 0 0.06 rpy=0 0 0
- added joint basefoot_peg_M2_basefoot_M2_joint_joint: type fixed, parent lowerleg_M2_link, child footM2_link, origin xyz=0 0 0.06 rpy=0 0 0
- added joint basefoot_peg_M3_basefoot_M3_joint_joint: type fixed, parent lowerleg_M3_link, child footM3_link, origin xyz=0 0 0.06 rpy=0 0 0
- added joint head_joint: type fixed, parent base_link, child head_link, origin xyz=0 0 0 rpy=0 0 0, axis 0 0 1
- added joint head_upperlegM1_joint: type revolute, parent head_link, child upperleg_M1_link, origin xyz=-0.02165 -0.0125 0.005 rpy=3.14159 0 -2.61799, axis 0 1 0, limit lower=-0.2 upper=0.2 effort=0.1 velocity=0.005
- added joint head_upperlegM2_joint: type revolute, parent head_link, child upperleg_M2_link, origin xyz=0.02165 -0.0125 0.005 rpy=3.14159 0 -0.523599, axis 0 1 0, limit lower=-0.2 upper=0.2 effort=0.1 velocity=0.005
- added joint head_upperlegM3_joint: type revolute, parent head_link, child upperleg_M3_link, origin xyz=0.0 0.0254 0.005 rpy=3.14159 0 1.579, axis 0 1 0, limit lower=-0.2 upper=0.2 effort=0.1 velocity=0.005
- added joint upperlegM1_lowerlegM1_joint: type revolute, parent upperleg_M1_link, child lowerleg_M1_link, origin xyz=0 0 0.06 rpy=0 0 0, axis 0 1 0, limit lower=-0.2 upper=0.2 effort=0.1 velocity=0.005
- added joint upperlegM2_lowerlegM2_joint: type revolute, parent upperleg_M2_link, child lowerleg_M2_link, origin xyz=0 0 0.06 rpy=0 0 0, axis 0 1 0, limit lower=-0.2 upper=0.2 effort=0.1 velocity=0.005
- added joint upperlegM3_lowerlegM3_joint: type revolute, parent upperleg_M3_link, child lowerleg_M3_link, origin xyz=0 0 0.06 rpy=0 0 0, axis 0 1 0, limit lower=-0.2 upper=0.2 effort=0.1 velocity=0.005
- joint world_joint: origin xyz=0 0 0.025 rpy=0 0 0 -> xyz=0 0 0 rpy=0 0 0

Commit message: wip

File: urdf/unit03/src/my_gurdy_description/urdf/gurdy.urdf (robot description, URDF)
Before this commit: robot gurdy, 12 links, 11 joints
Links:
- link base_link: mass None -> 0.01; geometry collision box size=0.01 0.01 0.01
- link footM1_link: mass None -> 0.01; geometry collision sphere radius=0.008; visual sphere radius=0.008
- link footM2_link: mass None -> 0.01; geometry collision sphere radius=0.008; visual sphere radius=0.008
- link footM3_link: mass None -> 0.01; geometry collision sphere radius=0.008; visual sphere radius=0.008
- link head_link: mass None -> 0.01; geometry collision cylinder length=0.04 radius=0.05; visual mesh filename=package://my_gurdy_description/models/gurdy/meshes/gurdy_he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
- link lowerleg_M1_link: mass None -> 0.01; geometry collision cylinder length=0.06 radius=0.0015; visual mesh filename=package://my_gurdy_description/models/gurdy/meshes/gurdy_lo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
- link lowerleg_M2_link: mass None -> 0.01; geometry collision cylinder length=0.06 radius=0.0015; visual mesh filename=package://my_gurdy_description/models/gurdy/meshes/gurdy_lo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
- link lowerleg_M3_link: mass None -> 0.01; geometry collision cylinder length=0.06 radius=0.0015; visual mesh filename=package://my_gurdy_description/models/gurdy/meshes/gurdy_lo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
- link upperleg_M1_link: mass None -> 0.01; geometry collision cylinder length=0.06 radius=0.0025; visual mesh filename=package://my_gurdy_description/models/gurdy/meshes/gurdy_hi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
- link upperleg_M2_link: mass None -> 0.01; geometry collision cylinder length=0.06 radius=0.0025; visual mesh filename=package://my_gurdy_description/models/gurdy/meshes/gurdy_hi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
- link upperleg_M3_link: mass None -> 0.01; geometry collision cylinder length=0.06 radius=0.0025; visual mesh filename=package://my_gurdy_description/models/gurdy/meshes/gurdy_hi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
Joints:
- joint head_upperlegM1_joint: limit lower=-0.2 upper=0.2 effort=0.1 velocity=0.005 -> lower=-0.2 upper=0.2 effort=1 velocity=0.005
- joint head_upperlegM2_joint: limit lower=-0.2 upper=0.2 effort=0.1 velocity=0.005 -> lower=-0.2 upper=0.2 effort=1 velocity=0.005
- joint head_upperlegM3_joint: limit lower=-0.2 upper=0.2 effort=0.1 velocity=0.005 -> lower=-0.2 upper=0.2 effort=1 velocity=0.005
- joint upperlegM1_lowerlegM1_joint: limit lower=-0.2 upper=0.2 effort=0.1 velocity=0.005 -> lower=-0.2 upper=0.2 effort=1 velocity=0.005
- joint upperlegM2_lowerlegM2_joint: limit lower=-0.2 upper=0.2 effort=0.1 velocity=0.005 -> lower=-0.2 upper=0.2 effort=1 velocity=0.005
- joint upperlegM3_lowerlegM3_joint: limit lower=-0.2 upper=0.2 effort=0.1 velocity=0.005 -> lower=-0.2 upper=0.2 effort=1 velocity=0.005

Commit message: gurdy seems to work

File: urdf/unit03/src/my_gurdy_description/urdf/gurdy.urdf (robot description, URDF)
Before this commit: robot gurdy, 12 links, 11 joints
Links:
- removed link world
Joints:
- removed joint world_joint
